File: LAB 1/KiCad/Lab1_KiCad/Lab1_KiCad.sch (KiCad schematic (older format))
At the start: 9 parts, among them U1 AT89C4051-12PU, Y1 12 MHz

Commit message: ready kicad scheme & pdf
Parts:
- added 10k: R_POT, symbol Device:R_POT
Connections:
- wire segments 33 -> 42
- no-connect marks 0 -> 7
Other:
- note removed: "LCD_E"
- note removed: "LCD_RS"
- note removed: "Potentiometer"
Changed lines of the file:
@@
 Wire Wire Line
 	6300 4150 5200 4150
-Wire Wire Line
-	6000 3250 6300 3250
-Text Notes 5700 3300 0    50   ~ 0
-LCD_RS
 $Comp
 L power:GND #PWR?
@@
 	0    1    1    0
 $EndComp
-Wire Wire Line
-	6300 2950 6000 2950
-Text Notes 5650 2950 0    50   ~ 0
-LCD_E
 $Comp
 L Device:C C5
@@
 $EndComp
 Wire Notes Line
-	7100 3000 7500 3000
-Wire Notes Line
-	7500 3000 7500 2900
-Wire Notes Line
-	7500 2900 7100 2900
-Wire Notes Line
 	7100 2900 7100 3000
-Text Notes 7100 3000 0    35   ~ 0
-Potentiometer
 $Comp
 L power:GND #PWR?
@@
 	1    0    0    -1
 $EndComp
+$Comp
+L Device:R_POT 10k
+U 1 1 60831499
+P 7450 2950
+F 0 "10k" H 7380 2904 50  0000 R CNN
+F 1 "R_POT" H 7380 2995 50  0000 R CNN
+F 2 "" H 7450 2950 50  0001 C CNN
+F 3 "~" H 7450 2950 50  0001 C CNN
+	1    7450 2950
+	-1   0    0    1
+$EndComp
+NoConn ~ 7100 3550
+NoConn ~ 7100 3650
+Wire Wire Line
+	7100 2950 7300 2950
+Wire Wire Line
+	7450 2800 7450 2550
+Wire Wire Line
+	7450 2550 6700 2550
+Wire Wire Line
+	7450 3100 7450 4350
+Wire Wire Line
+	7450 4350 6700 4350
+Connection ~ 6700 4350
+Wire Wire Line
+	5200 4450 5850 4450
+Wire Wire Line
+	5850 2950 6300 2950
+Wire Wire Line
+	5850 2950 5850 4450
+Wire Wire Line
+	5200 4350 5700 4350
+Wire Wire Line
+	5700 4350 5700 3250
+Wire Wire Line
+	5700 3250 6300 3250
+NoConn ~ 5200 4950
+NoConn ~ 5200 4850
+NoConn ~ 5200 4750
+NoConn ~ 5200 4650
+NoConn ~ 5200 4550
 $EndSCHEMATC
